File: PCB_Design/VGA_adapter/VGA_adapter.sch (KiCad schematic (older format))
At the start: 2 parts, among them J1 VGA Output, J2 PIC24 Curiosity Board Adapter

Commit message: PCB_Design: Add resistors to .sch and 3D model for pins
Parts:
- added R1, R2, R3: 470, Resistor_SMD:R_0805_2012Metric, symbol Device:R
Connections:
- wire segments 25 -> 30
Other:
- moved on the sheet: J1, J2
